File: Hardware/OpenBookReaderC v26.sch (EAGLE design)
At the start: 103 parts, among them IC1 BD5229G-TR, IC2 XC6220A331MR-G, J1 FH34SRJ-24S-0.5SH_99_, J2 SAMACSYS_PARTS_USB4110-GF-A, J3 QWIIC_RIGHT_ANGLE, J4 112A-TAAR-R03_ATTEND, Q1 SI1308EDL-T1-GE3, Q2 20V/4.2A/52mΩ/1.4W, Q3 20V/4.2A/52mΩ/1.4W, U1 W25Q512JVEIQ, U2 ESP32-C6-WROOM-1-N8, U3 DS3231SN#, U4 MAX17048G+T10

Commit message: s
Parts:
- C1, C10, C1_BAT, C1_BAT1, C1_BAT2, C2, C2_BAT, C3, C4_USB, C5, C5_USB, C6, C7, C8, C_DELAY, EPD_C1, EPD_C10, EPD_C11, EPD_C12, EPD_C2, EPD_C5, EPD_C6, EPD_C7, EPD_C8, EPD_C9: device DeskAssistant v19 v1:ESP32_WROVER_EAGLE-LTSPICE_CC0402 -> DeskAssistant v19 v1:ESP32_WROVER_EAGLE-LTSPICE_C
- D10, D11, D12, D6, D8, D9: value PGB1010603MR -> PGB1010603MRCOSMINEL1; device DeskAssistant v19 v1:PGB1010603MR -> DeskAssistant v19 v1:PGB1010603MRCOSMINEL1
- D3, D4, D5: value MBR0530 -> MBR0530COSMINEL2; device DeskAssistant v19 v1:MBR0530 -> DeskAssistant v19 v1:MBR0530COSMINEL2
- R3, R4: device DeskAssistant v19 v1:ESP32_WROVER_EAGLE-LTSPICE_RR0402 -> DeskAssistant v19 v1:ESP32_WROVER_EAGLE-LTSPICE_R
- TP1, TP10, TP11, TP12, TP13, TP14, TP15, TP16, TP17, TP2, TP3, TP4, TP5, TP6, TP7, TP8, TP9: value TPTP20R -> TP; device DeskAssistant v19 v1:TPTP20R -> DeskAssistant v19 v1:TP
