File: Hardware/OpenBookReaderC v34.brd (EAGLE design)
At the start: 170.2 x 114.3 mm, 103 parts, among them IC1 BD5229G-TR, IC2 XC6220A331MR-G, J1 FH34SRJ-24S-0.5SH_99_, J2 SAMACSYS_PARTS_USB4110-GF-A, J3 QWIIC_RIGHT_ANGLE, J4 112A-TAAR-R03_ATTEND, Q1 SI1308EDL-T1-GE3, Q2 20V/4.2A/52mΩ/1.4W, Q3 20V/4.2A/52mΩ/1.4W, U1 W25Q512JVEIQ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

Commit message: s
Parts:
- D10, D11, D12, D6, D8, D9: value PGB1010603MR -> PGB1010603MRCOSMINEL1
- D3, D4, D5: value MBR0530 -> MBR0530COSMINEL2
- TP1, TP10, TP11, TP12, TP13, TP14, TP15, TP16, TP17, TP2, TP3, TP4, TP5, TP6, TP7, TP8, TP9: value TPTP20R -> TP
Routing:
- net GND: track 674.7 -> 674.8 mm, vias 17 -> 105
